Commit message: add oak-d and sdf boxes on gz

File: delorian_ws/src/delorian_description/urdf/delorian_core.xacro (robot description, xacro)
@@ -114,5 +114,5 @@
         <parent link="oak_link"/>
         <child link="oak_optical_link"/>
-        <origin xyz="0 0 0" rpy="${-pi/2} 0 ${-pi/2}"/>
+        <origin xyz="0 0 0" rpy="${0} 0 ${0}"/>
     </joint>
 </robot>
