Commit message: cambios urdf gz y base, incluir oak

File: delorian_ws/src/delorian_description/urdf/delorian.gazebo.xacro (robot description, xacro)
@@ -34,3 +34,35 @@
         </plugin>
     </gazebo>
+    <gazebo reference="oak_link">
+        <sensor name="oak" type="rgbd_camera">
+            <topic>oak</topic>
+            <gz_frame_id>oak_optical_link</gz_frame_id>
+            <update_rate>30</update_rate>
+            <always_on>true</always_on>
+            <visualize>true</visualize>
+            <camera>
+                <horizontal_fov>1.2</horizontal_fov>
+                <image>
+                    <width>640</width>
+                    <height>400</height>
+                    <format>R8G8B8</format>
+                </image>
+                <clip>
+                    <near>0.2</near>
+                    <far>10</far>
+                </clip>
+                <depth_camera>
+                    <clip>
+                        <near>0.2</near>
+                        <far>10</far>
+                    </clip>
+                </depth_camera>
+                <noise>
+                    <type>gaussian</type>
+                    <mean>0</mean>
+                    <stddev>0.007</stddev>
+                </noise>
+            </camera>
+        </sensor>
+    </gazebo>
 </robot>

File: delorian_ws/src/delorian_description/urdf/delorian_core.xacro (robot description, xacro)
@@ -43,4 +43,7 @@
                 <mesh filename="package://delorian_description/meshes/main_frame.stl" scale="0.001 0.001 0.001"/>
             </geometry>
+            <material name="Metal">
+                <color rgba="0.3 0.3 0.3 1"/>
+            </material>
         </visual>
     </link>
@@ -69,4 +72,7 @@
                     <mesh filename="package://delorian_description/meshes/wheel.stl" scale="0.001 0.001 0.001"/>
                 </geometry>
+                <material name="Caucho rojo">
+                    <color rgba="0 0 0 1"/>
+                </material>
             </visual>
             <collision>
@@ -88,3 +94,25 @@
     <xacro:wheel name="front_right_wheel" x="${wheelbase/2}"  side="-1"/>
     <xacro:wheel name="rear_right_wheel"  x="${-wheelbase/2}" side="-1"/>
+    <link name="oak_link">
+        <visual>
+            <geometry>
+                <box size="0.03 0.10 0.04"/>
+            </geometry>
+            <material name="rosado-raro">
+                <color rgba="0.9 0.5 0.6 1"/>
+            </material>
+        </visual>
+    </link>
+    <joint name="oak_joint" type="fixed">
+        <parent link="base_link"/>
+        <child link="oak_link"/>
+        <origin xyz="0.335 0 0.30" rpy="0 0 0"/>
+    </joint>
+    <link name="oak_optical_link">
+    </link>
+    <joint name="oak_optical_joint" type="fixed">
+        <parent link="oak_link"/>
+        <child link="oak_optical_link"/>
+        <origin xyz="0 0 0" rpy="${-pi/2} 0 ${-pi/2}"/>
+    </joint>
 </robot>

Commit message: add imu and gps in gazebo and urdf core

File: delorian_ws/src/delorian_description/urdf/delorian.gazebo.xacro (robot description, xacro)
@@ -67,3 +67,19 @@
         </sensor>
     </gazebo>
+    <gazebo reference="imu_link">
+        <sensor name="imu" type="imu">
+            <topic>imu/data</topic>
+            <gz_frame_id>imu_link</gz_frame_id>
+            <update_rate>100</update_rate>
+            <always_on>true</always_on>
+        </sensor>
+    </gazebo>
+    <gazebo reference="gps_link">
+        <sensor name="navsat" type="navsat">
+            <topic>gps/fix</topic>
+            <gz_frame_id>gps_link</gz_frame_id>
+            <update_rate>10</update_rate>
+            <always_on>true</always_on>
+        </sensor>
+    </gazebo>
 </robot>

File: delorian_ws/src/delorian_description/urdf/delorian_core.xacro (robot description, xacro)
@@ -116,3 +116,17 @@
         <origin xyz="0 0 0" rpy="${0} 0 ${0}"/>
     </joint>
+    <!-- ===== IMU ===== -->
+    <link name="imu_link"/>
+    <joint name="imu_joint" type="fixed">
+        <parent link="base_link"/>
+        <child link="imu_link"/>
+        <origin xyz="0 0 0.05" rpy="0 0 0"/>
+    </joint>
+    <!-- ===== GPS (antena) ===== -->
+    <link name="gps_link"/>
+    <joint name="gps_joint" type="fixed">
+        <parent link="base_link"/>
+        <child link="gps_link"/>
+        <origin xyz="-0.15 0 0.35" rpy="0 0 0"/>
+    </joint>
 </robot>
